File: schematics/kicad/game.kicad_sch (KiCad schematic)
At the start: 5 parts, among them J1 2-Axis JoyStick

Commit message: update schematics
Connections:
- net LCD_EN: now also A1.22 (D7)
- net LCD_RS: now also A1.21 (D6)
Changed lines of the file:
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@@
+	(wire
+		(pts
+			(xy 147.32 82.55) (xy 147.32 91.44)
+		)
+		(stroke
+			(width 0)
+			(type default)
+		)
+	)
 	(wire
 		(pts
@@
 		(pts
 			(xy 165.1 91.44) (xy 165.1 82.55)
+		)
+		(stroke
+			(width 0)
+			(type default)
+		)
+	)
+	(wire
+		(pts
+			(xy 149.86 91.44) (xy 149.86 82.55)
 		)
 		(stroke
@@
 		(effects
 			(font
+				(size 1.27 1.27)
+			)
+			(justify left bottom)
+		)
+	)
+	(label "LCD_RS"
+		(at 147.32 91.44 90)
+		(effects
+			(font
+				(size 1.27 1.27)
+			)
+			(justify left bottom)
+		)
+	)
+	(label "LCD_EN"
+		(at 149.86 91.44 90)
+		(effects
+			(font
